Commit message: Fix mesh path in urdf

File: res/dora.urdf (robot description, URDF)
Before this commit: robot dora, 4 links, 3 joints
Links:
- link base_link: geometry collision mesh filename=dora_vaz.stl; visual mesh filename=dora_vaz.stl

Commit message: Remake urdf

File: res/dora.urdf (robot description, URDF)
Before this commit: robot dora, 4 links, 3 joints
Links:
- removed link wheel_1
- removed link wheel_2
- removed link wheel_3
- link base_link: geometry collision mesh filename=package://dora_urdf_rviz2/meshes/dora_vaz.stl scale=${body_scale_xyz}; visual mesh filename=package://dora_urdf_rviz2/meshes/dora_vaz.stl scale=${body_scale_xyz}
Joints:
- removed joint wheel_1_joint
- removed joint wheel_2_joint
- removed joint wheel_3_joint
