Commit message: Fix urdf, stl file locations

File: ros2_ws/src/controller/res/dora.urdf (robot description, URDF)
Before this commit: robot dora, 1 links, 0 joints
Links:
- link base_link: geometry collision mesh filename=package://controller/res/dora_vaz.stl scale=${body_scale_xyz}; visual mesh filename=package://controller/res/dora_vaz.stl scale=${body_scale_xyz}

Commit message: STL PLS

File: ros2_ws/src/controller/res/dora.urdf (robot description, URDF)
Before this commit: robot dora, 1 links, 0 joints
Links:
- link base_link: geometry collision mesh filename=file://$(find controller)/res/dora_vaz.stl scale=${body_scale_xyz}; visual mesh filename=file://$(find controller)/res/dora_vaz.stl scale=${body_scale_xyz}

Commit message: Visualisation base

File: ros2_ws/src/controller/res/dora.urdf (robot description, URDF)
Before this commit: robot dora, 1 links, 0 joints
Links:
- added link base_footprint
- added link lidar_link; collision cylinder length=${20*body_scale} radius=${40*body_scale}; visual cylinder length=${20*body_scale} radius=${40*body_scale}
- link base_link: geometry collision mesh filename=${mesh_path} scale=${body_scale_xyz}; visual mesh filename=${mesh_path} scale=${body_scale_xyz}
Joints:
- added joint base_joint: type fixed, parent base_link, child base_footprint, origin xyz=0 0 ${-body_height/10} rpy=0 0 0
- added joint lidar_joint: type fixed, parent base_link, child lidar_link, origin xyz=0 0 ${body_height*1.5}

Commit message: cleanup

File: ros2_ws/src/controller/res/dora.urdf (robot description, URDF)
Before this commit: robot dora, 3 links, 2 joints
Links:
- link lidar_link: geometry collision cylinder length=${lidar_length*body_scale} radius=${lidar_radius*body_scale}; visual cylinder length=${lidar_length*body_scale} radius=${lidar_radius*body_scale}
Joints:
- joint lidar_joint: origin xyz=0 0 ${body_height*1.5} -> xyz=0 0 ${body_height*lidar_distance}

Commit message: New WASD control started, mock_lidar for home testing started

File: ros2_ws/src/controller/res/dora.urdf (robot description, URDF)
Before this commit: robot dora, 3 links, 2 joints
Joints:
- joint base_joint: child base_footprint -> base_link; origin xyz=0 0 ${-body_height/10} rpy=0 0 0 -> xyz=0 0 ${body_height/20} rpy=0 0 0; parent base_link -> base_footprint

Commit message: Fix uart receive

File: ros2_ws/src/controller/res/dora.urdf (robot description, URDF)
Before this commit: robot dora, 1 links, 0 joints
Links:
- added link base_lidar
- link base_link: geometry collision mesh filename=${mesh_path} scale=${mesh_scale}; visual mesh filename=${mesh_path} scale=${mesh_scale}
Joints:
- added joint lidar_joint: type fixed, parent base_link, child base_lidar, origin xyz=0 0 ${body_to_floor + body_height + lidar_height}

Commit message: dumpit

File: ros2_ws/src/controller/res/dora.urdf (robot description, URDF)
Before this commit: robot dora, 1 links, 0 joints
Links:
- added link camera1
- added link camera2
- added link cameras_center
- added link laser
- link base_link: geometry collision mesh filename=${mesh_path} scale=${mesh_scale}; visual mesh filename=${mesh_path} scale=${mesh_scale}
Joints:
- added joint camera1_joint: type fixed, parent cameras_center, child camera1, origin xyz=0 ${-cam_to_cam_dist * 0.5} 0
- added joint camera2_joint: type fixed, parent cameras_center, child camera2, origin xyz=0 ${cam_to_cam_dist * 0.5} 0
- added joint camera_center_joint: type fixed, parent base_link, child cameras_center, origin xyz=${cos(camera_angle) * cam_to_center_dist} ${sin(camera_angle) * cam_to_center_dist} ${body_to_floor + cam_height} rpy=0 0 ${camera_angle}
- added joint lidar_joint: type fixed, parent base_link, child laser, origin xyz=0 0 ${body_to_floor + body_height + lidar_height}
